File: MCU.kicad_sch (KiCad schematic)
At the start: 18 parts, among them J1 Conn_ARM_JTAG_SWD_10, J4 Conn_ARM_JTAG_SWD_10, J5 UART, U2 STM32F030C8T6, Y1 8Mhz

Commit message: updated part sizes for pick and place
Parts:
- C2, C3, C4, C6, C8: # (none) -> C14663; Height (none) -> .8; Length (none) -> 1.6; Tape (none) -> 8x4; Width (none) -> .8
- C5, C7: # (none) -> C1634; Height (none) -> .8; Length (none) -> 1.6; Tape (none) -> 8x4; Width (none) -> .8
- J1, J4: # (none) -> C6332249
- J5: # (none) -> C2691448
- R2, R3, R4, R5: # (none) -> C25804; Height (none) -> .45; Length (none) -> 1.6; Tape (none) -> 8x4; Width (none) -> .8
- SW3: LCSC (none) -> C319392
- SW4: Field9 2.3 -> (none); LCSC (none) -> C319392; Length (none) -> 2.3
- U2: # (none) -> C23922; Height (none) -> 1.45; Length (none) -> 7; Tape (none) -> 16x12; Width (none) -> 7
- Y1: # (none) -> C648984; Height (none) -> .65; Length (none) -> 3.2; Width (none) -> 2.5
