File: driver.kicad_sch (KiCad schematic)
At the start: 9 parts, among them J2 PEEL_MOTOR, J3 Conn_01x06_Socket, U5 DRV8837, U6 DRV8837

Commit message: updated part sizes for pick and place
Parts:
- C14, C15, C16, C17: # (none) -> C14663; Height (none) -> .8; Length (none) -> 1.6; Tape (none) -> 8x4; Width (none) -> .8
- J2: # (none) -> C2845379; Height (none) -> 3.5; Length (none) -> 7.5; Tape (none) -> 16x8; Width (none) -> 5
- J3: # (none) -> C2845383; Height (none) -> 3.5; Length (none) -> 12.5; Tape (none) -> 24x8; Width (none) -> 5
- R13: # (none) -> C25804; Height (none) -> .45; Length (none) -> 1.6; Tape (none) -> 8x4; Width (none) -> .8
- U5, U6: # (none) -> C191000; Height (none) -> .8; Length (none) -> 2; Tape (none) -> 8x4; Width (none) -> 2
