File: power.kicad_sch (KiCad schematic)
At the start: 14 parts, among them U3 AMS1117-3.3, U4 MC34063AD

Commit message: updated part sizes for pick and place
Parts:
- C10, C9: # (none) -> C7432785; Height (none) -> 1.6; Length (none) -> 3.2; Tape (none) -> 8x4; Width (none) -> 1.6
- C11: # (none) -> C2836442; Height (none) -> 7.7; Length (none) -> 6.3; Tape (none) -> 16x8; Width (none) -> 6.3
- C12: # (none) -> C107092; Height (none) -> .8; Length (none) -> 1.6; Tape (none) -> 8x4; Width (none) -> .8
- C13: # (none) -> C5354997; Height (none) -> 7.7; Length (none) -> 6.3; Tape (none) -> 16x8; Width (none) -> 6.3
- D4: # (none) -> C965804; Height (none) -> .4; Length (none) -> 1.6; Tape (none) -> 8x4; Width (none) -> .8
- D5: # (none) -> C82544; Height (none) -> 1; Length (none) -> 3.65; Tape (none) -> 8x4; Width (none) -> 1.55
- L1: # (none) -> C467145; Height (none) -> 4.5; Length (none) -> 6; Tape (none) -> 12x8; Width (none) -> 6
- R10: # (none) -> C2934265; Height (none) -> .6; Length (none) -> 2; Tape (none) -> 8x4; Width (none) -> 1.25
- R11: # (none) -> C114627; Height (none) -> .45; Length (none) -> 1.6; Tape (none) -> 8x4; Width (none) -> .8
- R12: # (none) -> C163424; Height (none) -> .45; Length (none) -> 1.6; Tape (none) -> 8x4; Width (none) -> .8
- R9: # (none) -> C21190; Height (none) -> .45; Length (none) -> 1.6; Tape (none) -> 8x4; Width (none) -> .8
- U3: # (none) -> C347222; Height (none) -> 1.8; Length (none) -> 3.5; Tape (none) -> 12x8; Width (none) -> 6
- U4: # (none) -> C80213; Height (none) -> 1.5; Length (none) -> 4.9; Tape (none) -> 12x8; Width (none) -> 3.9
